Commit message: add omniwheels

File: description/macros/base.xacro (robot description, xacro)
@@ -6,38 +6,119 @@
 	<link name="origin_link"/>
 	<link name="base_link">
-	<inertial>
-		<mass value="0.07862944645"/>
-		<inertia
-			ixx="0.00002035985530754"
-			ixy="0"
-			ixz="0"
-			iyy="0.00002035985530754"
-			iyz="0"
-			izz="0.00003945961663220"/>
-	</inertial>
-  <visual>
-    <geometry>
-      <box size="0.3 0.3 0.01"/>
-    </geometry>
-    <origin rpy="0 0 0" xyz="0 0 0"/>
-    <material name="red"/>
-  </visual>
-	<collision>
+		<inertial>
+			<mass value="0.07862944645"/>
+			<inertia
+				ixx="0.00002035985530754"
+				ixy="0"
+				ixz="0"
+				iyy="0.00002035985530754"
+				iyz="0"
+				izz="0.00003945961663220"/>
+		</inertial>
+	  <visual>
+	    <geometry>
+	      <box size="0.3 0.3 0.01"/>
+	    </geometry>
+	    <origin rpy="0 0 0" xyz="0 0 0"/>
+	    <material name="red"/>
+	  </visual>
+		<collision>
 		<geometry>
       <box size="0.3 0.3 0.01"/>
 		</geometry>
 	</collision>
-	</link>
-	<joint
-		name="base_joint"
-		type="fixed">
-		<parent link="origin_link" />
-		<child link="base_link" />
-		<origin xyz="0 0 0"/>
-	</joint>
+		</link>
+  <joint name="origin_joint" type="fixed">
+      <parent link="origin_link"/>
+      <child link="base_link"/>
+      <origin xyz="0 0 0.065"/>
+  </joint>
+	<!--front left wheel and motor-->
+  <link name="front_left_motor">
+      <visual>
+        <geometry>
+          <cylinder length="0.145" radius="0.015"/>
+        </geometry>
+        <origin rpy="0 0 0" xyz="0 0 0"/>
+        <material name="blue"/>
+      </visual>
+  </link>
+  <joint name="base_to_front_left_motor" type="fixed">
+      <parent link="base_link"/>
+      <child link="front_left_motor"/>
+      <origin rpy="0 1.570796 0.785398" xyz="0.07 0.07 -0.035" />
+  </joint>
 	<xacro:rim_macro
-		name="left"
-		color="0.3 0 0"
-		xyz="0 0 0"
-		rpy="0 0 0"/>
+			name="front_left"
+			color="1 1 1"
+			xyz="0 0 0.0875"
+			rpy="0 0 0"
+			parent_link="front_left_motor"
+	/>
+<!--front right wheel and motor-->
+	<link name="front_right_motor">
+		    <visual>
+		      <geometry>
+		        <cylinder length="0.145" radius="0.015"/>
+		      </geometry>
+		      <origin rpy="0 0 0" xyz="0 0 0"/>
+		      <material name="blue"/>
+		    </visual>
+		</link>
+	<joint name="base_to_front_right_motor" type="fixed">
+		    <parent link="base_link"/>
+		    <child link="front_right_motor"/>
+		    <origin rpy="0 1.570796 -0.785398" xyz="0.07 -0.07 -0.035" />
+		</joint>
+	<xacro:rim_macro
+			name="front_right"
+			color="1 1 1"
+			xyz="0 0 0.0875"
+			rpy="0 0 0"
+			parent_link="front_right_motor"
+	 />
+<!--back left wheel and motor-->
+<link name="back_right_motor">
+    <visual>
+      <geometry>
+        <cylinder length="0.145" radius="0.015"/>
+      </geometry>
+      <origin rpy="0 0 0" xyz="0 0 0"/>
+      <material name="blue"/>
+    </visual>
+</link>
+<joint name="base_to_back_right_motor" type="fixed">
+    <parent link="base_link"/>
+    <child link="back_right_motor"/>
+    <origin rpy="0 1.570796 3.92699" xyz="-0.07 -0.07 -0.035" />
+</joint>
+<xacro:rim_macro
+		name="back_right"
+		color="1 1 1"
+		xyz="0 0 0.0875"
+		rpy="0 0 0"
+		parent_link="back_right_motor"
+ />
+<!--back left wheel and motor-->
+<link name="back_left_motor">
+    <visual>
+      <geometry>
+        <cylinder length="0.145" radius="0.015"/>
+      </geometry>
+      <origin rpy="0 0 0" xyz="0 0 0"/>
+      <material name="blue"/>
+    </visual>
+</link>
+<joint name="base_to_back_left_motor" type="fixed">
+    <parent link="base_link"/>
+    <child link="back_left_motor"/>
+    <origin rpy="0 1.570796 2.35619" xyz="-0.07 0.07 -0.035" />
+</joint>
+<xacro:rim_macro
+		name="back_left"
+		color="1 1 1"
+		xyz="0 0 0.0875"
+		rpy="0 0 0"
+		parent_link="back_left_motor"
+ />
 </robot>

File: description/macros/rim.xacro (robot description, xacro)
@@ -4,5 +4,5 @@
 	<xacro:macro
 		name="rim_macro"
-		params="name color xyz rpy">
+		params="name color xyz rpy parent_link">
 		<link name="rim_${name}_link">
 			<inertial>
@@ -20,5 +20,5 @@
 			<visual>
 				<geometry>
-					<mesh filename="package://description/mesh/wheelasm.stl"/>
+					<mesh filename="package://description/mesh/wheelasm.stl" scale="0.001 0.001 0.001"/>
 				</geometry>
 				<material name="rim_${name}_material">
@@ -28,5 +28,5 @@
 			<collision>
 				<geometry>
-					<mesh filename="package://description/mesh/wheelasm.stl"/>
+					<mesh filename="package://description/mesh/wheelasm.stl" scale="0.001 0.001 0.001"/>
 				</geometry>
 			</collision>
@@ -34,7 +34,6 @@
 		<joint
 			name="rim_${name}_joint"
-			type="continuous"
-		>
-			<parent link="base_link" />
+			type="continuous">
+			<parent link="${parent_link}" />
 			<child link="rim_${name}_link" />
 			<axis xyz="0 0 1"/>
@@ -45,7 +44,52 @@
 		<xacro:roller_macro
 			parent="${name}"
-			name="one"
-			xyz="0.01355 0 0.0055"
-			rpy="-1.570796326794896 0 0"/>
-	</xacro:macro>
+			name="front_left"
+			xyz="0 -0.024 0.0065"
+			rpy="0 -${pi/2} 0"/>
+	<xacro:roller_macro
+		parent="${name}"
+		name="back_right"
+		xyz="0 0.024 -0.0065"
+		rpy="0 -${pi/2} 0"/>
+	<xacro:roller_macro
+		parent="${name}"
+		name="front_top_right"
+		xyz="-0.0141068 0.0194164 0.0065"
+		rpy="0 -${pi/2} ${pi/5}"/>
+<xacro:roller_macro
+	parent="${name}"
+	name="front_down_right"
+	xyz="0.0141068 0.0194164 0.0065"
+	rpy="0 -${pi/2} -${pi/5}"/>
+	<xacro:roller_macro
+		parent="${name}"
+		name="back_top_left"
+		xyz="-0.0141068 -0.0194164 -0.0065"
+		rpy="0 -${pi/2} -${pi/5}"/>
+<xacro:roller_macro
+	parent="${name}"
+	name="back_down_left"
+	xyz="0.0141068 -0.0194164 -0.0065"
+	rpy="0 -${pi/2} ${pi/5}"/>
+	<xacro:roller_macro
+		parent="${name}"
+		name="front_top_left"
+		xyz="-0.0228254 -0.0074164 0.0065"
+		rpy="0 -${pi/2} ${3*pi/5}"/>
+		<xacro:roller_macro
+			parent="${name}"
+			name="front_down_left"
+			xyz="0.0228254 -0.0074164 0.0065"
+			rpy="0 -${pi/2} -${3*pi/5}"/>
+		<xacro:roller_macro
+			parent="${name}"
+			name="back_down_right"
+			xyz="0.0228254 0.0074164 -0.0065"
+			rpy="0 -${pi/2} ${3*pi/5}"/>
+			<xacro:roller_macro
+				parent="${name}"
+				name="back_top_right"
+				xyz="-0.0228254 0.0074164 -0.0065"
+				rpy="0 -${pi/2} -${3*pi/5}"/>
+</xacro:macro>
 </robot>

File: description/macros/roller.xacro (robot description, xacro)
@@ -17,6 +17,7 @@
 			</inertial>
 			<visual>
+				<origin rpy="0 -${pi/2} 0" xyz="0 0 0"/>
 				<geometry>
-					<mesh filename="package://description/mesh/rubberwheel.stl"/>
+					<mesh filename="package://description/mesh/rubberwheel.stl" scale="0.001 0.001 0.001"/>
 				</geometry>
 				<material name="roller_material">
@@ -26,5 +27,5 @@
 			<collision>
 				<geometry>
-					<mesh filename="package://description/mesh/rubberwheel.stl"/>
+					<mesh filename="package://description/mesh/rubberwheel.stl" scale="0.001 0.001 0.001"/>
 				</geometry>
 			</collision>
